File: _autosave-UART.sch (KiCad schematic (older format))
At the start: 12 parts, among them P3 CONN_01X04, P5 CONN_01X04, P6 CONN_01X04, U4 MAX3227

Commit message: review and discussion done
Parts:
- gave numbers to parts that had none: 3
Connections:
- net GND: now also U7.2 (GND)
Changed lines of the file:
@@
 	5750 3550 5750 3650
 $Comp
-L mechanical-connectors:CONN_01X03 P?
+L mechanical-connectors:CONN_01X03 P2
 U 1 1 5FE08D5C
 P 6150 3450
-F 0 "P?" H 6228 3536 50  0000 L CNN
+F 0 "P2" H 6228 3536 50  0000 L CNN
 F 1 "CONN_01X03" H 6228 3445 50  0000 L CNN
 F 2 "CON_wuerth:WR-TBL_691322310003" H 6228 3354 50  0000 L CNN
@@
 $EndComp
 $Comp
-L mechanical-connectors:CONN_01X03 P?
+L mechanical-connectors:CONN_01X03 P10
 U 1 1 5FE14388
 P 6500 5400
-F 0 "P?" H 6578 5486 50  0000 L CNN
+F 0 "P10" H 6578 5486 50  0000 L CNN
 F 1 "CONN_01X03" H 6578 5395 50  0000 L CNN
 F 2 "CON_wuerth:WR-TBL_691322310003" H 6578 5304 50  0000 L CNN
@@
 $EndComp
 $Comp
-L CAN-transceiver:SN65HVD232 U?
+L CAN-transceiver:SN65HVD232 U7
 U 1 1 5FE154CA
 P 4700 5700
-F 0 "U?" H 5225 6587 60  0000 C CNN
+F 0 "U7" H 5225 6587 60  0000 C CNN
 F 1 "SN65HVD232" H 5225 6481 60  0000 C CNN
 F 2 "SOIC:SOIJ-8_5.3x5.3mm_Pitch1.27mm" H 5550 5650 60  0001 C CNN
@@
 	6300 5500 6100 5500
 $Comp
-L power-supply:GND #PWR?
+L power-supply:GND #PWR0151
 U 1 1 5FE1EAD5
 P 6100 5600
-AR Path="/5FCC65EC/5FE1EAD5" Ref="#PWR?"  Part="1"
+AR Path="/5FCC65EC/5FE1EAD5" Ref="#PWR0151"  Part="1"
 AR Path="/600B38DA/5FE1EAD5" Ref="#PWR?"  Part="1"
-F 0 "#PWR?" H 6100 5350 50  0001 C CNN
+F 0 "#PWR0151" H 6100 5350 50  0001 C CNN
 F 1 "GND" H 6105 5427 50  0000 C CNN
 F 2 "" H 6100 5600 50  0000 C CNN
@@
 NoConn ~ 5750 5150
 NoConn ~ 5750 5550
+Wire Wire Line
+	4700 5550 4500 5550
+$Comp
+L power-supply:GND #PWR?
+U 1 1 5FD53433
+P 4500 5650
+AR Path="/5FCC65EC/5FD53433" Ref="#PWR?"  Part="1"
+AR Path="/600B38DA/5FD53433" Ref="#PWR?"  Part="1"
+F 0 "#PWR?" H 4500 5400 50  0001 C CNN
+F 1 "GND" H 4505 5477 50  0000 C CNN
+F 2 "" H 4500 5650 50  0000 C CNN
+F 3 "" H 4500 5650 50  0000 C CNN
+	1    4500 5650
+	1    0    0    -1
+$EndComp
+Wire Wire Line
+	4500 5550 4500 5650
 $EndSCHEMATC
