File: power.sch (KiCad schematic (older format))
At the start: 20 parts, among them P5 WR-TBL_691322310002, U4 TPS54335A

Commit message: somehow done with general layouting
Parts:
- added D1: TVS, diodes:DO-214AB, symbol devices:TVS
Connections:
- net +BATT: now also D1.1
- net GND: now also D1.2
Changed lines of the file:
@@
 Connection ~ 5950 1900
 Wire Wire Line
-	4550 2550 5250 2550
+	4550 2550 4850 2550
 Wire Wire Line
-	4550 1900 5250 1900
+	4550 1900 4850 1900
 Wire Wire Line
 	5250 1900 5950 1900
@@
 	1    0    0    -1
 $EndComp
+$Comp
+L devices:TVS D1
+U 1 1 5FD478B4
+P 4850 2200
+F 0 "D1" V 4759 2288 50  0000 L CNN
+F 1 "TVS" V 4850 2288 50  0000 L CNN
+F 2 "diodes:DO-214AB" V 4941 2288 50  0000 L CNN
+F 3 "" H 4850 2200 50  0000 C CNN
+	1    4850 2200
+	0    1    1    0
+$EndComp
+Connection ~ 4850 1900
+Wire Wire Line
+	4850 1900 5250 1900
+Wire Wire Line
+	4850 2500 4850 2550
+Connection ~ 4850 2550
+Wire Wire Line
+	4850 2550 5250 2550
 $EndSCHEMATC
