File: kicad_source/UART.sch (KiCad schematic (older format))
At the start: 15 parts, among them P10 CONN_01X03, P11 CONN_01X02, P2 CONN_01X03, P3 CONN_01X04, P5 CONN_01X04, P6 CONN_01X04, U4 MAX3227, U7 SN65HVD232

Commit message: tested and fixed last bugs
Parts:
- U7: footprint SOIC:SOIJ-8_5.3x5.3mm_Pitch1.27mm -> SOIC:SOIC-8_3.9x4.9mm_Pitch1.27mm
Changed lines of the file:
@@
 F 0 "U7" H 5225 6587 60  0000 C CNN
 F 1 "SN65HVD232" H 5225 6481 60  0000 C CNN
-F 2 "SOIC:SOIJ-8_5.3x5.3mm_Pitch1.27mm" H 5550 5650 60  0001 C CNN
+F 2 "SOIC:SOIC-8_3.9x4.9mm_Pitch1.27mm" H 5550 5650 60  0001 C CNN
 F 3 "" H 4700 5850 60  0000 C CNN
 	1    4700 5700
